Commit message: Created core URDF

File: description/robot_core.xacro (robot description, xacro)
@@ -1,4 +1,5 @@
 <?xml version="1.0"?>
 <robot xmlns:xacro="http://www.ros.org/wiki/xacro" >
+    <xacro:include filename="inertial_macros.xacro" />
     <material name="white">
         <color rgba="1 1 1 1" />
@@ -30,10 +31,19 @@
             <material name="white" />
         </visual>
+        <collision>
+            <origin xyz="0.15 0 0.075" />
+            <geometry>
+                <box size="0.3 0.3 0.15" />
+            </geometry>
+        </collision>
+        <xacro:inertial_box mass="0.5" x="0.3" y="0.3" z="0.15">
+            <origin xyz="0.15 0 0.075" rpy="0 0 0"/>
+        </xacro:inertial_box>
     </link>
     <!-- LEFT WHEEL LINK -->
-    <joint name="left wheel_joint" type="continuous" >
+    <joint name="left_wheel_joint" type="continuous" >
         <parent link="base_link"/>
-        <child link="left wheel_link" />
-        <origin xyz="0 0.175 0" rpy="${-pi/2} 0 0" />
+        <child link="left_wheel" />
+        <origin xyz="0 0.175 0" rpy="-${pi/2} 0 0" />
         <axis xyz="0 0 1"/>
     </joint>
@@ -45,8 +55,17 @@
             <material name="blue"/>
         </visual>
+        <collision>
+            <geometry>
+                <cylinder radius="0.05" length="0.04"/>
+            </geometry>
+        </collision>
+        <xacro:inertial_cylinder mass="0.1" length="0.04" radius="0.05">
+            <origin xyz="0 0 0" rpy="0 0 0"/>
+        </xacro:inertial_cylinder>
+    </link>
     <!-- RIGHT WHEEL LINK -->
-    <joint name="right wheel_joint" type="continuous" >
+    <joint name="right_wheel_joint" type="continuous" >
         <parent link="base_link"/>
-        <child link="right wheel_link" />
+        <child link="right_wheel" />
         <origin xyz="0 -0.175 0" rpy="${pi/2} 0 0" />
         <axis xyz="0 0 -1"/>
@@ -59,3 +78,35 @@
             <material name="blue"/>
         </visual>
+        <collision>
+            <geometry>
+                <cylinder radius="0.05" length="0.04"/>
+            </geometry>
+        </collision>
+        <xacro:inertial_cylinder mass="0.1" length="0.04" radius="0.05">
+            <origin xyz="0 0 0" rpy="0 0 0"/>
+        </xacro:inertial_cylinder>
+    </link>
+    <!-- CASTER WHEEL LINK -->
+    <joint name="caster_wheel_joint" type="fixed" >
+        <parent link="chassis"/>
+        <child link="caster_wheel" />
+        <origin xyz="0.24 0 0"  />
+        <axis xyz="0 0 -1"/>
+    </joint>
+    <link name="caster_wheel">
+        <visual>
+            <geometry>
+                <sphere radius="0.05"/>
+            </geometry>
+            <material name="black"/>
+        </visual>
+        <collision>
+            <geometry>
+                <sphere radius="0.05"/>
+            </geometry>
+        </collision>
+        <xacro:inertial_sphere mass="0.1" radius="0.05">
+            <origin xyz="0 0 0" rpy="0 0 0"/>
+        </xacro:inertial_sphere>
+    </link>
 </robot>

Commit message: gazebo_simulation

File: description/robot_core.xacro (robot description, xacro)
@@ -41,4 +41,7 @@
         </xacro:inertial_box>
     </link>
+    <gazebo reference="chassis">
+        <material>Gazebo/White</material>
+    </gazebo>
     <!-- LEFT WHEEL LINK -->
     <joint name="left_wheel_joint" type="continuous" >
@@ -64,4 +67,7 @@
         </xacro:inertial_cylinder>
     </link>
+   <gazebo reference="left_wheel">
+        <material>Gazebo/Blue</material>
+    </gazebo>
     <!-- RIGHT WHEEL LINK -->
     <joint name="right_wheel_joint" type="continuous" >
@@ -87,4 +93,7 @@
         </xacro:inertial_cylinder>
     </link>
+   <gazebo reference="right_wheel">
+        <material>Gazebo/Blue</material>
+    </gazebo>
     <!-- CASTER WHEEL LINK -->
     <joint name="caster_wheel_joint" type="fixed" >
@@ -110,3 +119,8 @@
         </xacro:inertial_sphere>
     </link>
+   <gazebo reference="caster_wheel">
+        <material>Gazebo/Black</material>
+        <mu1 value="0.001"/>
+        <mu2 value="0.001"/>
+    </gazebo>
 </robot>
